File: Earendel-1/_restore_backup_2026-06-11T09-59-47-708/Earendel-1.kicad_sch (KiCad schematic)
At the start: 37 parts, among them J1 SAMTEC-CES-110-01-X-D, J2 DS1021-1X2SF162-B, J3 78938-403HLF, J4 85_SMA-50-0-144_111_YH, U1 ATA8510-GHQW, U2 STM32F411CCUx, Y1 XRCGB24M000F0G00R0, Y2 CAA-4.000-18-3050-X

Commit message: Save State for PCB
Parts:
- removed TP1: TestPoint, Connector_Pin:Pin_D0.7mm_L6.5mm_W1.8mm_FlatFork, symbol Connector:TestPoint
- removed TP2, TP3, TP4, TP5, TP6, TP7, TP8: TestPoint, Connector_Pin:Pin_D0.9mm_L10.0mm_W2.4mm_FlatFork, symbol Connector:TestPoint
- C1, C10, C11, C12, C13, C14, C2, C3, C4, C5, C6, C7, C8, C9: footprint Capacitor_SMD:C_0805_2012Metric_Pad1.18x1.45mm_HandSolder -> Capacitor_SMD:C_0805_2012Metric
- J1: footprint Connector_Coaxial:SMA_Samtec_SMA-J-P-H-ST-EM1_EdgeMount -> SAMTEC-CES-110-01-X-D:SAMTEC-CES-110-01-X-D
- J2: footprint DS1021-1X2SF162-B:CONNFLY_DS1021-1X2SF162-B -> (none)
- L1, L2, L3: footprint Inductor_SMD:L_0805_2012Metric_Pad1.05x1.20mm_HandSolder -> Inductor_SMD:L_12x12mm_H8mm
- R1, R2, R3: footprint Resistor_SMD:R_0805_2012Metric_Pad1.20x1.40mm_HandSolder -> Resistor_SMD:R_0805_2012Metric
Connections:
- net AVCC is gone; now on net VDD: C4.1, U1.12 (AVCC)
- net DVCC is gone; now on net VDD: C6.1, U1.20 (DVCC)
- net VS_PA is gone; now on net VDD: C3.1, U1.8 (VS_PA)
- net CLK_OUT: no longer U2.32 (PA11)
Other:
- note added: "AVCC"
- note added: "DVCC"
- note added: "VS_PA"
