File: Earendel-1/Earendel-1.kicad_sch (KiCad schematic)
At the start: 37 parts, among them J1 SAMTEC-CES-110-01-X-D, J2 DS1021-1X2SF162-B, J3 78938-403HLF, J4 85_SMA-50-0-144_111_YH, U1 ATA8510-GHQW, U2 STM32F411CCUx, Y1 XRCGB24M000F0G00R0, Y2 CAA-4.000-18-3050-X

Commit message: commiting new libraries
Parts:
- removed J1: SAMTEC-CES-110-01-X-D, Connector_Coaxial:SMA_Samtec_SMA-J-P-H-ST-EM1_EdgeMount, symbol SAMTEC-CES-110-01-X-D:SAMTEC-CES-110-01-X-D
- removed J2: DS1021-1X2SF162-B, DS1021-1X2SF162-B:CONNFLY_DS1021-1X2SF162-B, symbol DS1021-1X2SF162-B:DS1021-1X2SF162-B
- removed J3: 78938-403HLF, 78938-403HLF:AMPHENOL_78938-403HLF, symbol 78938-403HLF:78938-403HLF
- added C15: 4.7uF, symbol Device:C
- added J1: MTMM-101-15-G-D-105, MTMM-101-15-G-D-105:SAMTEC_MTMM-101-15-G-D-105, symbol MTMM-101-15-G-D-105:MTMM-101-15-G-D-105
- added J2: TSW-101-05-T-T, TSW-101-05-T-T:SAMTEC_TSW-101-05-T-T, symbol TSW-101-05-T-T:TSW-101-05-T-T
- added J5: TSS-110-01-G-D, TSS-110-01-G-D:SAMTEC_TSS-110-01-G-D, symbol TSS-110-01-G-D:TSS-110-01-G-D
Connections:
- net DVCC: now also J5.01
- net GND: now also U2.8 (VSSA), C15.2, J1.02, J2.03, J5.04, J5.06, J5.08, J5.10, J5.12, J5.14, J5.16, J5.18, J5.20
- net JTCLK: now also J5.09
- net JTDI: now also J5.05
- net JTDO: now also J5.13
- net JTMS: now also J5.07
- net NJTRST: now also J5.03
- net NRST: now also J5.15
- net RX: now also J2.02
- net TX: now also J2.01
- net V+: now also J1.01
- net VDD: now also U2.9 (VDDA)
- net VCAP: now reaches U2.22 (VCAP1)
- net VCAP: now also C15.1

Commit message: first Routing
Parts:
- added J6: TSS-110-01-G-D, TSS-110-01-G-D:SAMTEC_TSS-110-01-G-D, symbol TSS-110-01-G-D:TSS-110-01-G-D
Connections:
- net CLK_OUT: now also J6.01
- net GND: now also J6.15
- net MISO: now also J6.07
- net MOSI: now also J6.09
- net NSS: now also J6.03
- net SCK: now also J6.05
- net LORA_CS: now reaches U2.33 (PA12)
- net SCL: now reaches U2.42 (PB6)
- net SCL: now also J6.11
- net SDA: now reaches U2.43 (PB7)
- net SDA: now also J6.13

Commit message: Programmer and ATA mostly routed
Parts:
- C15: footprint (none) -> Capacitor_SMD:C_0504_1310Metric_Pad0.83x1.28mm_HandSolder
- Y2: footprint CAA-4.000-18-3050-X:XTAL_CAA-4.000-18-3050-X -> CAA-4.000-18-3050-X-R(1):XTAL_CAA-4.000-18-3050-X-R
Connections:
- net JTRST is gone; now on net NJTRST: U2.40 (PB4)
- net SCK_2: now reaches U2.26 (PB13)
- net MISO_2: now reaches U2.27 (PB14)
- net MOSI_2: now reaches U2.28 (PB15)
Changed lines of the file:
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@@
 	(wire
 		(pts
+			(xy 177.8 119.38) (xy 186.69 119.38)
+		)
+		(stroke
+			(width 0)
+			(type default)
+		)
+	)
+	(wire
+		(pts
 			(xy 238.76 237.49) (xy 251.46 237.49)
 		)
@@
 	(wire
 		(pts
+			(xy 177.8 116.84) (xy 186.69 116.84)
+		)
+		(stroke
+			(width 0)
+			(type default)
+		)
+	)
+	(wire
+		(pts
 			(xy 222.25 73.66) (xy 227.33 73.66)
 		)
@@
 	(wire
 		(pts
+			(xy 177.8 114.3) (xy 186.69 114.3)
+		)
+		(stroke
+			(width 0)
+			(type default)
+		)
+	)
+	(wire
+		(pts
 			(xy 177.8 91.44) (xy 186.69 91.44)
 		)
@@
 		)
 	)
-	(label "JTRST"
+	(label "NJTRST"
 		(at 177.8 93.98 0)
 		(effects
@@
 		)
 	)
+	(label "MOSI_2"
+		(at 177.8 119.38 0)
+		(effects
+			(font
+				(size 1.27 1.27)
+			)
+			(justify left bottom)
+		)
+	)
 	(label "TX"
 		(at 227.33 78.74 0)
@@
 		)
 	)
+	(label "MISO_2"
+		(at 177.8 116.84 0)
+		(effects
+			(font
+				(size 1.27 1.27)
+			)
+			(justify left bottom)
+		)
+	)
 	(label "RX"
 		(at 283.21 180.34 0)
@@
 		)
 	)
+	(label "SCK_2"
+		(at 177.8 114.3 0)
+		(effects
+			(font
+				(size 1.27 1.27)
+			)
+			(justify left bottom)
+		)
+	)
 	(label "AVCC"
 		(at 35.56 153.67 0)
@@
 			)
 		)
-		(property "Footprint" ""
+		(property "Footprint" "Capacitor_SMD:C_0504_1310Metric_Pad0.83x1.28mm_HandSolder"
 			(at 155.9052 132.08 0)
 			(hide yes)
@@
 			)
 		)
-		(property "Footprint" "CAA-4.000-18-3050-X:XTAL_CAA-4.000-18-3050-X"
+		(property "Footprint" "CAA-4.000-18-3050-X-R(1):XTAL_CAA-4.000-18-3050-X-R"
 			(at 50.8 248.92 0)
 			(hide yes)

Commit message: Programmer and ATA mostly routed
Connections:
- net CLK_OUT: no longer J6.01
Changed lines of the file:
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@@
-	(wire
-		(pts
-			(xy 326.39 128.27) (xy 335.28 128.27)
-		)
-		(stroke
-			(width 0)
-			(type default)
-		)
-	)
 	(wire
 		(pts
@@
 		(effects
 			(font
-				(size 1.27 1.27)
-			)
-			(justify left bottom)
-		)
-	)
-	(label "CLK_OUT"
-		(at 326.39 128.27 0)
-		(effects
-			(font
