File: Earendel-1/_restore_backup_2026-06-27T19-08-24-010/Earendel-1.kicad_pcb (KiCad board)
At the start: 2 copper layers, 40 parts, among them J1 MTMM-101-15-G-D-105, J2 TSW-101-05-T-T, J4 85_SMA-50-0-144_111_YH, J5 TSS-110-01-G-D, J6 TSS-110-01-G-D, U1 ATA8510-GHQW, U2 STM32F411CCUx, Y1 XRCGB24M000F0G00R0, Y2 CAA-4.000-18-3050-X

Commit message: toying with traces
Parts:
- removed C16: C, Capacitor_SMD:C_0805_2012Metric_Pad1.18x1.45mm_HandSolder
- moved C5 98.7 mm to (128.5, 142.0)
- moved C4 89.3 mm to (128.5, 139.0), turned to 0 degrees
- moved C12 0.68 mm to (52.5, 91.0)
Connections:
- C3 pad 1: /VDD -> /VS_PA
- C4 pad 1: /VDD -> /AVCC
- C6 pad 1: /VDD -> /DVCC
- U1 pad 12: /VDD -> /AVCC
- U1 pad 20: /VDD -> /DVCC
- U1 pad 8: /VDD -> /VS_PA
Routing:
- net /VDD: track 77.4 -> 54.8 mm
- net /VS_PA: track 0.00 -> 6.77 mm
- net Net-(C7-Pad2): track 5.19 -> 0.00 mm
- net /ANT: track 5.02 -> 0.00 mm
- net Net-(C10-Pad1): track 4.85 -> 0.00 mm
- net /Wake_Up: track 15.5 -> 14.6 mm
- net GND: track 0.58 -> 0.00 mm
