File: Earendel-1/_restore_backup_2026-06-27T19-08-24-010/Earendel-1.kicad_sch (KiCad schematic)
At the start: 40 parts, among them J1 MTMM-101-15-G-D-105, J2 TSW-101-05-T-T, J4 85_SMA-50-0-144_111_YH, J5 TSS-110-01-G-D, J6 TSS-110-01-G-D, U1 ATA8510-GHQW, U2 STM32F411CCUx, Y1 XRCGB24M000F0G00R0, Y2 CAA-4.000-18-3050-X

Commit message: toying with traces
Parts:
- removed C16: C, Capacitor_SMD:C_0805_2012Metric_Pad1.18x1.45mm_HandSolder, symbol Device:C
- C15: footprint Capacitor_SMD:C_0805_2012Metric_Pad1.18x1.45mm_HandSolder -> Capacitor_SMD:C_0504_1310Metric_Pad0.83x1.28mm_HandSolder
Connections:
- net DVCC: now also C6.1, U1.20 (DVCC)
- net VDD: no longer C3.1, C4.1, C6.1, U1.12 (AVCC), U1.20 (DVCC), U1.8 (VS_PA)
- new net AVCC: C4.1, U1.12 (AVCC)
- new net VS_PA: C3.1, U1.8 (VS_PA)
Changed lines of the file:
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@@
 		)
 	)
-	(label "VDD"
+	(label "DVCC"
 		(at 116.84 115.57 0)
 		(effects
@@
 		)
 	)
-	(label "VDD"
+	(label "AVCC"
 		(at 36.83 110.49 0)
 		(effects
@@
 		)
 	)
-	(label "VDD"
+	(label "VS_PA"
 		(at 25.4 153.67 0)
 		(effects
@@
 		)
 	)
-	(label "VDD"
+	(label "DVCC"
 		(at 55.88 153.67 0)
 		(effects
@@
 		)
 	)
-	(label "VDD"
+	(label "AVCC"
 		(at 35.56 153.67 0)
 		(effects
@@
 		)
 	)
-	(label "VDD"
+	(label "VS_PA"
 		(at 36.83 100.33 0)
 		(effects
@@
 		)
 	)
-	(label "VDD"
-		(at 236.22 39.37 0)
-		(effects
-			(font
-				(size 1.27 1.27)
-			)
-			(justify left bottom)
-		)
-	)
 	(label "CLK_OUT"
 		(at 116.84 110.49 0)
@@
 			)
 		)
-		(property "Footprint" "Capacitor_SMD:C_0805_2012Metric_Pad1.18x1.45mm_HandSolder"
+		(property "Footprint" "Capacitor_SMD:C_0504_1310Metric_Pad0.83x1.28mm_HandSolder"
 			(at 155.9052 132.08 0)
 			(hide yes)
@@
 	)
 	(symbol
-		(lib_id "power:GND")
-		(at 236.22 46.99 0)
-		(unit 1)
-		(body_style 1)
-		(exclude_from_sim no)
-		(in_bom yes)
-		(on_board yes)
-		(in_pos_files yes)
-		(dnp no)
-		(fields_autoplaced yes)
-		(property "Reference" "#PWR017"
-			(at 236.22 53.34 0)
-			(hide yes)
-			(show_name no)
-			(do_not_autoplace no)
-			(effects
-				(font
-					(size 1.27 1.27)
-				)
-			)
-		)
-		(property "Value" "GND"
-			(at 236.22 52.07 0)
-			(show_name no)
-			(do_not_autoplace no)
-			(effects
-				(font
-					(size 1.27 1.27)
-				)
-			)
-		)
-		(property "Footprint" ""
-			(at 236.22 46.99 0)
-			(hide yes)
-			(show_name no)
-			(do_not_autoplace no)
-			(effects
-				(font
-					(size 1.27 1.27)
-				)
-			)
-		)
-		(property "Datasheet" ""
-			(at 236.22 46.99 0)
-			(hide yes)
-			(show_name no)
-			(do_not_autoplace no)
-			(effects
-				(font
-					(size 1.27 1.27)
-				)
-			)
-		)
-		(property "Description" "Power symbol creates a global label with name \"GND\" , ground"
-			(at 236.22 46.99 0)
-			(hide yes)
-			(show_name no)
-			(do_not_autoplace no)
-			(effects
-				(font
-					(size 1.27 1.27)
-				)
-			)
-		)
-		(pin "1"
-		)
-		(instances
-			(project "Earendel-1"
-				(path "/80bbe4cb-c454-49fe-926e-47095f357e2d"
-					(reference "#PWR017")
-					(unit 1)
-				)
-			)
-		)
-	)
-	(symbol
 		(lib_id "Device:C")
 		(at 462.28 77.47 0)
@@
 					(unit 1)
 				)
-			)
-		)
-	)
-	(symbol
-		(lib_id "Device:C")
-		(at 236.22 43.18 0)
-		(unit 1)
-		(body_style 1)
-		(exclude_from_sim no)
-		(in_bom yes)
-		(on_board yes)
-		(in_pos_files yes)
-		(dnp no)
-		(fields_autoplaced yes)
-		(property "Reference" "C16"
-			(at 240.03 41.9099 0)
-			(show_name no)
-			(do_not_autoplace no)
-			(effects
-				(font
-					(size 1.27 1.27)
-				)
-				(justify left)
-			)
-		)
-		(property "Value" "C"
-			(at 240.03 44.4499 0)
-			(show_name no)
-			(do_not_autoplace no)
-			(effects
-				(font
-					(size 1.27 1.27)
-				)
-				(justify left)
-			)
-		)
-		(property "Footprint" "Capacitor_SMD:C_0805_2012Metric_Pad1.18x1.45mm_HandSolder"
-			(at 237.1852 46.99 0)
-			(hide yes)
-			(show_name no)
-			(do_not_autoplace no)
-			(effects
-				(font
-					(size 1.27 1.27)
-				)
-			)
-		)
-		(property "Datasheet" ""
-			(at 236.22 43.18 0)
-			(hide yes)
-			(show_name no)
-			(do_not_autoplace no)
-			(effects
-				(font
-					(size 1.27 1.27)
-				)
-			)
-		)
-		(property "Description" "Unpolarized capacitor"
-			(at 236.22 43.18 0)
-			(hide yes)
-			(show_name no)
-			(do_not_autoplace no)
-			(effects
-				(font
-					(size 1.27 1.27)
-				)
-			)
-		)
-		(pin "2"
-		)
-		(pin "1"
-		)
-		(instances
-			(project "Earendel-1"
-				(path "/80bbe4cb-c454-49fe-926e-47095f357e2d"
-					(reference "C16")
-					(unit 1)
-				)
