File: Earendel-1/_restore_backup_2026-06-28T17-56-12-651/Earendel-1.kicad_pcb (KiCad board)
At the start: 2 copper layers, 40 parts, among them J1 MTMM-101-15-G-D-105, J2 TSW-101-05-T-T, J4 85_SMA-50-0-144_111_YH, J5 TSS-110-01-G-D, J6 TSS-110-01-G-D, U1 ATA8510-GHQW, U2 STM32F411CCUx, Y1 XRCGB24M000F0G00R0, Y2 CAA-4.000-18-3050-X

Commit message: Finished V0 PCB
Parts:
- C15: footprint Capacitor_SMD:C_0805_2012Metric_Pad1.18x1.45mm_HandSolder -> Capacitor_SMD:C_0504_1310Metric_Pad0.83x1.28mm_HandSolder
- moved R3 85.6 mm to (144.5, 126.8)
- moved R1 78.2 mm to (144.5, 120.9), turned to 0 degrees
- moved C6 73.0 mm to (133.3, 130.0), turned to 0 degrees
- moved R2 71.5 mm to (144.5, 123.9)
- moved TP8 70.0 mm to (136.9, 107.1)
- moved TP4 66.3 mm to (132.5, 107.1)
- moved TP3 61.3 mm to (132.5, 103.2)
- moved TP6 55.5 mm to (136.9, 99.4)
- moved TP2 52.6 mm to (132.5, 99.4)
- moved TP5 46.9 mm to (132.5, 110.9)
- moved TP7 44.1 mm to (136.9, 103.2)
- moved C5 8.11 mm to (42.5, 93.5), turned to 0 degrees
- moved C15 1.60 mm to (53.6, 95.5)
Connections:
- R2 pad 2: /DVCC -> /MCU_VDD
- U2 pad 26: unconnected-(U2-PB13-Pad26) -> /SCK_2
- U2 pad 27: unconnected-(U2-PB14-Pad27) -> /MISO_2
- U2 pad 28: unconnected-(U2-PB15-Pad28) -> /MOSI_2
Routing:
- net GND: track 65.6 -> 0.58 mm, vias 18 -> 0
- net /VDD: track 135.1 -> 77.4 mm, vias 6 -> 4
- net /IRQ: track 21.1 -> 0.00 mm, vias 4 -> 0
- net /DVCC: track 20.5 -> 0.00 mm, vias 1 -> 0
- net /JTDI: track 31.7 -> 21.0 mm
- net /NRST: track 67.1 -> 58.7 mm
- net /SCK: track 41.3 -> 34.6 mm, vias 3 -> 2
- net /MOSI: track 42.7 -> 36.2 mm
- net /BOOT0: track 5.97 -> 0.00 mm
- net /SDA: track 35.5 -> 38.5 mm
- net /VCAP: track 9.33 -> 7.17 mm
Other:
- board text removed: "+"
- board text removed: "-"
- board text removed: "Designed by Joshua Leevers"
- board text removed: "GFSK APRS Radio Board"
- board text removed: "GND"
- board text removed: "PRG_HDR"
- board text removed: "Rx"
- board text removed: "Tx"
