File: Earendel-1/_restore_backup_2026-06-28T17-56-12-651/Earendel-1.kicad_sch (KiCad schematic)
At the start: 40 parts, among them J1 MTMM-101-15-G-D-105, J2 TSW-101-05-T-T, J4 85_SMA-50-0-144_111_YH, J5 TSS-110-01-G-D, J6 TSS-110-01-G-D, U1 ATA8510-GHQW, U2 STM32F411CCUx, Y1 XRCGB24M000F0G00R0, Y2 CAA-4.000-18-3050-X

Commit message: Finished V0 PCB
Connections:
- net SCK_2: now reaches U2.26 (PB13)
- net MISO_2: now reaches U2.27 (PB14)
- net MOSI_2: now reaches U2.28 (PB15)
Changed lines of the file:
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@@
+	(wire
+		(pts
+			(xy 177.8 119.38) (xy 186.69 119.38)
+		)
+		(stroke
+			(width 0)
+			(type default)
+		)
+	)
 	(wire
 		(pts
@@
 	(wire
 		(pts
+			(xy 177.8 116.84) (xy 186.69 116.84)
+		)
+		(stroke
+			(width 0)
+			(type default)
+		)
+	)
+	(wire
+		(pts
 			(xy 222.25 73.66) (xy 227.33 73.66)
 		)
@@
 		(pts
 			(xy 222.25 88.9) (xy 227.33 88.9)
+		)
+		(stroke
+			(width 0)
+			(type default)
+		)
+	)
+	(wire
+		(pts
+			(xy 177.8 114.3) (xy 186.69 114.3)
 		)
 		(stroke
@@
 		)
 	)
+	(label "MOSI_2"
+		(at 177.8 119.38 0)
+		(effects
+			(font
+				(size 1.27 1.27)
+			)
+			(justify left bottom)
+		)
+	)
 	(label "TX"
 		(at 227.33 78.74 0)
@@
 		)
 	)
+	(label "MISO_2"
+		(at 177.8 116.84 0)
+		(effects
+			(font
+				(size 1.27 1.27)
+			)
+			(justify left bottom)
+		)
+	)
 	(label "RX"
 		(at 283.21 180.34 0)
@@
 		(effects
 			(font
+				(size 1.27 1.27)
+			)
+			(justify left bottom)
+		)
+	)
+	(label "SCK_2"
+		(at 177.8 114.3 0)
+		(effects
+			(font
